File: hardware/BM64_Breakout/BM64_Breakout.sch (KiCad schematic (older format))
At the start: 28 parts, among them J1 USB_B_Micro, J2 Conn_02x03_Odd_Even, J3 Conn_02x03_Odd_Even, J4 Conn_01x02, J5 Conn_01x01, J6 Conn_01x08, J7 Conn_01x07, J8 Conn_02x02_Odd_Even, U1 MIC803, U2 BM64SPKS1MC1

Commit message: Updated from Mac
Parts:
- D1, D2: footprint LED_SMD:LED_0603_1608Metric -> Diode_SMD:D_0603_1608Metric
Changed lines of the file:
@@
 $EndDescr
-$Comp
-L bm64:BM64SPKS1MC1 U2
-U 1 1 5BBADDC3
-P 5550 2000
-F 0 "U2" H 6750 2290 60  0000 C CNN
-F 1 "BM64SPKS1MC1" H 6750 2184 60  0000 C CNN
-F 2 "BM64:BM64_Module" H 5550 2000 50  0001 C CNN
-F 3 "" H 5550 2000 50  0001 C CNN
-	1    5550 2000
-	1    0    0    -1
-$EndComp
 $Comp
 L Device:LED D1
@@
 F 0 "D1" V 8188 1633 50  0000 R CNN
 F 1 "LED" V 8097 1633 50  0000 R CNN
-F 2 "LED_SMD:LED_0603_1608Metric" H 8150 1750 50  0001 C CNN
+F 2 "Diode_SMD:D_0603_1608Metric" H 8150 1750 50  0001 C CNN
 F 3 "~" H 8150 1750 50  0001 C CNN
 	1    8150 1750
@@
 F 0 "D2" V 8588 1633 50  0000 R CNN
 F 1 "LED" V 8497 1633 50  0000 R CNN
-F 2 "LED_SMD:LED_0603_1608Metric" H 8550 1750 50  0001 C CNN
+F 2 "Diode_SMD:D_0603_1608Metric" H 8550 1750 50  0001 C CNN
 F 3 "~" H 8550 1750 50  0001 C CNN
 	1    8550 1750
@@
 Wire Wire Line
 	1500 2700 2050 2700
+$Comp
+L bm64:BM64SPKS1MC1 U2
+U 1 1 5BF6120F
+P 5550 2000
+F 0 "U2" H 6750 2290 60  0000 C CNN
+F 1 "BM64SPKS1MC1" H 6750 2184 60  0000 C CNN
+F 2 "BM64:BM64_Module" H 5550 2000 50  0001 C CNN
+F 3 "" H 5550 2000 50  0001 C CNN
+	1    5550 2000
+	1    0    0    -1
+$EndComp
 $EndSCHEMATC
